Commit message: sensors add

File: description/robot.urdf.xacro (robot description, xacro)
@@ -2,3 +2,5 @@
 <robot xmlns:xacro="http://www.ros.org/wiki/xacro"  name="robot">
     <xacro:include filename="robot_core.xacro" />
+    <xacro:include filename="gazebo_control.xacro" />
+     <xacro:include filename="lidar.xacro" />
 </robot>

File: description/robot_core.xacro (robot description, xacro)
@@ -4,4 +4,7 @@
     <material name="white">
         <color rgba="1 1 1 1" />
+    </material>
+     <material name="red">
+        <color rgba="1 0 0 1" />
     </material>
     <material name="orange">
@@ -42,4 +45,9 @@
         </xacro:inertial_box>
     </link>
+    <gazebo reference = "chasis">
+        <material>
+            Gazebo/white
+        </material>
+    </gazebo>
     <!-- LEFT WHEEL LINK -->
     <joint name="left_wheel_joint" type="continuous">
@@ -66,4 +74,9 @@
         </xacro:inertial_cylinder>
     </link>
+   <gazebo reference = "left_wheel">
+        <material>
+            Gazebo/Blue
+        </material>
+    </gazebo>
     <!-- RIGHT WHEEL LINK -->
     <joint name="right_wheel_joint" type="continuous">
@@ -90,4 +103,9 @@
         </xacro:inertial_cylinder>
     </link>
+     <gazebo reference = "right_wheel">
+        <material>
+            Gazebo/Blue
+        </material>
+    </gazebo>
     <!-- CASTER WHEEL -->
     <joint name="caster_wheel_joint" type="fixed">
@@ -113,3 +131,10 @@
         </xacro:inertial_sphere>
     </link>
+     <gazebo reference = "caster_wheel">
+        <material>
+            Gazebo/Black
+        </material>
+        <mu1 value = "0.001"/>
+        <mu2 value = "0.001"/>
+      </gazebo>
 </robot>
